File: PCB/KiCad_Project/WAR_Button.kicad_pcb (KiCad board)
At the start: 2 copper layers, 17.3 x 34.8 mm, 22 parts, among them IC1 ATTINY84A-M, P1 USB_OTG, P2 BATT, P3 HEADER, P4 T3, P5 T2, P6 T4, P7 T0, P8 T1, Q1 MCP73831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

Commit message: Added MOSFET
Parts:
- added C4: 1uF, Capacitors_SMD:C_0603, F.Cu at (149.2, 91.4)
- added Q2: NTR2101PT1G, Housings_SOT-23_SOT-143_TSOT-6:SOT-23, F.Cu at (151.9, 91.3)
- added R5: 100K, Resistors_SMD:R_0603, F.Cu at (151.9, 88.8)
- P4: value T3 -> T2
- P5: value T2 -> T1
- P6: value T4 -> T3
- P7: value T0 -> T4
- P8: value T1 -> T0
Connections:
- BLE1 pad 17: BATT_VCC -> LOAD_VCC
- BLE1 pad 27: BATT_VCC -> LOAD_VCC
- C1 pad 1: PROG_VCC -> USB_VCC
- C3 pad 2: BATT_VCC -> LOAD_VCC
- IC1 pad 5: BATT_VCC -> LOAD_VCC
- IC1 pad 9: BATT_VCC -> LOAD_VCC
- P1 pad 1: PROG_VCC -> USB_VCC
- P3 pad 2: PROG_VCC -> LOAD_VCC
- Q1 pad 4: PROG_VCC -> USB_VCC
- R1 pad 1: PROG_VCC -> USB_VCC
Routing:
- net LOAD_VCC: track 0.00 -> 47.3 mm, vias 0 -> 3
- net PROG_VCC: track 38.3 -> 0.00 mm, vias 1 -> 0
- net USB_VCC: track 0.00 -> 36.2 mm, vias 0 -> 1
- net BATT_VCC: track 61.1 -> 37.9 mm, vias 2 -> 1
- net PROG_GND: track 108.7 -> 121.1 mm
- net Net-(P1-Pad6): track 12.4 -> 13.4 mm
Other:
- board size 17.3 x 34.8 mm -> 17 x 34.5 mm

Commit message: Added GERBER and Drill files
Parts:
- renumbered P8 to T0, P5 to T1, P4 to T2, P6 to T3, P7 to T4
Changed lines of the file:
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@@
     (links 76)
     (no_connects 3)
-    (area 142.545999 59.741999 159.714001 94.436001)
+    (area 139.363 59.809499 164.319191 96.987)
     (thickness 1.6)
     (drawings 4)
@@
     (visible_elements 7FFFFF7F)
     (pcbplotparams
-      (layerselection 0x00030_80000001)
-      (usegerberextensions false)
+      (layerselection 0x010f0_80000001)
+      (usegerberextensions true)
       (excludeedgelayer true)
       (linewidth 0.100000)
@@
       (outputformat 1)
       (mirror false)
-      (drillshape 1)
+      (drillshape 0)
       (scaleselection 1)
       (outputdirectory ""))
@@
     (descr "Mesurement Point, Square, SMD Pad,  1.5mm x 1.5mm,")
     (tags "Mesurement Point, Square, SMD Pad, 1.5mm x 1.5mm,")
-    (fp_text reference P4 (at 0 3.81) (layer B.SilkS) hide
-      (effects (font (size 1 1) (thickness 0.15)) (justify mirror))
-    )
-    (fp_text value T2 (at -2.54 0.127) (layer B.Fab)
+    (fp_text reference T2 (at -2.54 0) (layer B.SilkS)
+      (effects (font (size 1 1) (thickness 0.15)) (justify mirror))
+    )
+    (fp_text value T2 (at -2.54 0.127) (layer B.Fab) hide
       (effects (font (size 1 1) (thickness 0.15)) (justify mirror))
     )
@@
     (descr "Mesurement Point, Square, SMD Pad,  1.5mm x 1.5mm,")
     (tags "Mesurement Point, Square, SMD Pad, 1.5mm x 1.5mm,")
-    (fp_text reference P5 (at 0 3.81) (layer B.SilkS) hide
-      (effects (font (size 1 1) (thickness 0.15)) (justify mirror))
-    )
-    (fp_text value T1 (at -3.302 0) (layer B.Fab)
+    (fp_text reference T1 (at -3.429 0) (layer B.SilkS)
+      (effects (font (size 1 1) (thickness 0.15)) (justify mirror))
+    )
+    (fp_text value T1 (at -3.302 0) (layer B.Fab) hide
       (effects (font (size 1 1) (thickness 0.15)) (justify mirror))
     )
@@
     (descr "Mesurement Point, Square, SMD Pad,  1.5mm x 1.5mm,")
     (tags "Mesurement Point, Square, SMD Pad, 1.5mm x 1.5mm,")
-    (fp_text reference P6 (at 0 3.81) (layer B.SilkS) hide
-      (effects (font (size 1 1) (thickness 0.15)) (justify mirror))
-    )
-    (fp_text value T3 (at -1.905 0) (layer B.Fab)
+    (fp_text reference T3 (at -1.905 0) (layer B.SilkS)
+      (effects (font (size 1 1) (thickness 0.15)) (justify mirror))
+    )
+    (fp_text value T3 (at -1.905 0) (layer B.Fab) hide
       (effects (font (size 1 1) (thickness 0.15)) (justify mirror))
     )
@@
     (descr "Mesurement Point, Square, SMD Pad,  1.5mm x 1.5mm,")
     (tags "Mesurement Point, Square, SMD Pad, 1.5mm x 1.5mm,")
-    (fp_text reference P7 (at -4.7625 -2.4765) (layer F.SilkS) hide
-      (effects (font (size 1 1) (thickness 0.15)))
-    )
-    (fp_text value T4 (at 1.905 0) (layer F.Fab)
+    (fp_text reference T4 (at 1.905 0) (layer F.SilkS)
+      (effects (font (size 1 1) (thickness 0.15)))
+    )
+    (fp_text value T4 (at 1.905 0) (layer F.Fab) hide
       (effects (font (size 1 1) (thickness 0.15)))
     )
@@
     (descr "Mesurement Point, Square, SMD Pad,  1.5mm x 1.5mm,")
     (tags "Mesurement Point, Square, SMD Pad, 1.5mm x 1.5mm,")
-    (fp_text reference P8 (at 0 3.81) (layer B.SilkS) hide
-      (effects (font (size 1 1) (thickness 0.15)) (justify mirror))
-    )
-    (fp_text value T0 (at -2.159 0) (layer B.Fab)
-      (effects (font (size 1 1) (thickness 0.15)) (justify mirror))
-    )
+    (fp_text reference T0 (at -1.905 0.127) (layer B.SilkS)
+      (effects (font (size 1 1) (thickness 0.15)) (justify mirror))
+    )
+    (fp_text value T0 (at -2.159 0) (layer B.Fab) hide
+      (effects (font (size 1 1) (thickness 0.15)) (justify mirror))
+    )
