File: PCB/KiCad_Project/WAR_Button.sch (KiCad schematic (older format))
At the start: 8 parts, among them IC1 ATTINY84A-MM, SW1 SW_PUSH, SW2 SW_PUSH

Commit message: Updated Schematic
Parts:
- removed P?: CONN_01X04, symbol CONN_01X04
- removed R1: 100K, symbol R_Small
- removed SW2: SW_PUSH, symbol SW_PUSH
- added D?: LED, symbol LED
- added P?: CONN_01X06, symbol CONN_01X06
- added R?: R_Small, symbol R_Small
Connections:
- net labels added: P1, P2, P3, P4, PROG_GND, PROG_VIN, WAKE
- wire segments 21 -> 31
Other:
- moved on the sheet: BT1
Changed lines of the file:
@@
-$EndComp
-$Comp
-L R_Small R1
-U 1 1 560D7942
-P 10550 5050
-F 0 "R1" H 10580 5070 50  0000 L CNN
-F 1 "100K" H 10580 5010 50  0000 L CNN
-F 2 "" H 10550 5050 60  0000 C CNN
-F 3 "" H 10550 5050 60  0000 C CNN
-	1    10550 5050
-	1    0    0    -1
-$EndComp
-$Comp
-L GND #PWR10
-U 1 1 560D7A93
-P 10550 5300
-F 0 "#PWR10" H 10550 5050 50  0001 C CNN
-F 1 "GND" H 10550 5150 50  0000 C CNN
-F 2 "" H 10550 5300 60  0000 C CNN
-F 3 "" H 10550 5300 60  0000 C CNN
-	1    10550 5300
-	1    0    0    -1
 $EndComp
 $Comp
@@
 $EndComp
 $Comp
-L SW_PUSH SW2
-U 1 1 560D8A92
-P 3900 4450
-F 0 "SW2" H 4050 4560 50  0000 C CNN
-F 1 "SW_PUSH" H 3900 4370 50  0000 C CNN
-F 2 "" H 3900 4450 60  0000 C CNN
-F 3 "" H 3900 4450 60  0000 C CNN
-	1    3900 4450
-	1    0    0    -1
-$EndComp
-$Comp
-L GND #PWR5
-U 1 1 560D8AC0
-P 4350 4450
-F 0 "#PWR5" H 4350 4200 50  0001 C CNN
-F 1 "GND" H 4350 4300 50  0000 C CNN
-F 2 "" H 4350 4450 60  0000 C CNN
-F 3 "" H 4350 4450 60  0000 C CNN
-	1    4350 4450
-	0    -1   -1   0
-$EndComp
-$Comp
 L Battery BT1
 U 1 1 560D9989
-P 5250 3650
-F 0 "BT1" H 5350 3700 50  0000 L CNN
-F 1 "Battery" H 5350 3600 50  0000 L CNN
-F 2 "" V 5250 3690 60  0000 C CNN
-F 3 "" V 5250 3690 60  0000 C CNN
-	1    5250 3650
+P 6350 3900
+F 0 "BT1" H 6450 3950 50  0000 L CNN
+F 1 "Battery" H 6450 3850 50  0000 L CNN
+F 2 "" V 6350 3940 60  0000 C CNN
+F 3 "" V 6350 3940 60  0000 C CNN
+	1    6350 3900
 	1    0    0    -1
 $EndComp
@@
 L GND #PWR7
 U 1 1 560D9BA1
-P 5250 3800
-F 0 "#PWR7" H 5250 3550 50  0001 C CNN
-F 1 "GND" H 5250 3650 50  0000 C CNN
-F 2 "" H 5250 3800 60  0000 C CNN
-F 3 "" H 5250 3800 60  0000 C CNN
-	1    5250 3800
+P 6350 4250
+F 0 "#PWR7" H 6350 4000 50  0001 C CNN
+F 1 "GND" H 6350 4100 50  0000 C CNN
+F 2 "" H 6350 4250 60  0000 C CNN
+F 3 "" H 6350 4250 60  0000 C CNN
+	1    6350 4250
 	1    0    0    -1
 $EndComp
@@
 L +3V3 #PWR6
 U 1 1 560D9BC3
-P 5250 3500
-F 0 "#PWR6" H 5250 3350 50  0001 C CNN
-F 1 "+3V3" H 5250 3640 50  0000 C CNN
-F 2 "" H 5250 3500 60  0000 C CNN
-F 3 "" H 5250 3500 60  0000 C CNN
-	1    5250 3500
+P 6350 3550
+F 0 "#PWR6" H 6350 3400 50  0001 C CNN
+F 1 "+3V3" H 6350 3690 50  0000 C CNN
+F 2 "" H 6350 3550 60  0000 C CNN
+F 3 "" H 6350 3550 60  0000 C CNN
+	1    6350 3550
 	1    0    0    -1
 $EndComp
@@
 	8550 4350 8850 4350
 Wire Wire Line
-	10550 4850 10550 4950
-Wire Wire Line
-	10550 5150 10550 5300
-Wire Wire Line
 	4200 4200 4350 4200
 Wire Wire Line
 	3600 4200 3150 4200
-Wire Wire Line
-	4200 4450 4350 4450
-Wire Wire Line
-	3600 4450 3600 4300
-Wire Wire Line
-	3600 4300 3150 4300
 Text GLabel 10750 3350 2    60   Input ~ 0
 BLE_TX
@@
 Wire Wire Line
 	10550 3450 10750 3450
+Text GLabel 4100 3400 2    60   Input ~ 0
+BLE_RX
+Text GLabel 4100 3550 2    60   Input ~ 0
+BLE_TX
+Wire Wire Line
+	3150 3400 4100 3400
+Wire Wire Line
+	3150 3500 4100 3500
+Wire Wire Line
+	4100 3500 4100 3550
 Wire Wire Line
 	3150 3300 3700 3300
 Wire Wire Line
-	3150 3400 3450 3400
-Wire Wire Line
-	3450 3400 3450 3300
-Connection ~ 3450 3300
-$Comp
-L CONN_01X04 P?
-U 1 1 560DD29E
-P 2250 2150
-F 0 "P?" H 2250 2400 50  0000 C CNN
-F 1 "CONN_01X04" V 2350 2150 50  0000 C CNN
-F 2 "" H 2250 2150 60  0000 C CNN
-F 3 "" H 2250 2150 60  0000 C CNN
-	1    2250 2150
+	3550 3600 3150 3600
+Text GLabel 3550 3600 2    60   Input ~ 0
+WAKE
+Text GLabel 10550 4850 2    60   Input ~ 0
+WAKE
+Text GLabel 2850 1950 3    60   Input ~ 0
+P1
+Text GLabel 2950 1950 3    60   Input ~ 0
+P2
+Text GLabel 3050 1950 3    60   Input ~ 0
+P3
+Text GLabel 3150 1950 3    60   Input ~ 0
+P4
+$Comp
+L CONN_01X06 P?
+U 1 1 561F3005
+P 2900 1750
+F 0 "P?" H 2900 2100 50  0000 C CNN
+F 1 "CONN_01X06" V 3000 1750 50  0000 C CNN
+F 2 "" H 2900 1750 60  0000 C CNN
+F 3 "" H 2900 1750 60  0000 C CNN
+	1    2900 1750
 	0    -1   -1   0
 $EndComp
+Text GLabel 2600 2250 3    60   Input ~ 0
+PROG_VIN
+Text GLabel 2750 2250 3    60   Input ~ 0
+PROG_GND
+Wire Wire Line
+	2750 1950 2750 2250
+Wire Wire Line
+	2600 2250 2600 1950
+Wire Wire Line
+	2600 1950 2650 1950
+Text GLabel 6100 4100 3    60   Input ~ 0
+PROG_GND
+Wire Wire Line
+	6100 4100 6100 4050
+Wire Wire Line
+	6100 4050 6350 4050
+Wire Wire Line
+	6350 4050 6350 4250
+Text GLabel 6100 3650 1    60   Input ~ 0
+PROG_VIN
+Wire Wire Line
+	6100 3650 6100 3750
+Wire Wire Line
+	6100 3750 6350 3750
+Wire Wire Line
+	6350 3750 6350 3550
+Text GLabel 3150 3700 2    60   Input ~ 0
+P1
+Text GLabel 3150 3800 2    60   Input ~ 0
+P2
+Text GLabel 3150 3900 2    60   Input ~ 0
+P3
+Text GLabel 3150 4500 2    60   Input ~ 0
+P4
+$Comp
+L LED D?
+U 1 1 561F3B46
+P 4100 3850
+F 0 "D?" H 4100 3950 50  0000 C CNN
+F 1 "LED" H 4100 3750 50  0000 C CNN
+F 2 "" H 4100 3850 60  0000 C CNN
+F 3 "" H 4100 3850 60  0000 C CNN
+	1    4100 3850
+	-1   0    0    1
+$EndComp
+$Comp
+L R_Small R?
+U 1 1 561F3B97
+P 3650 3850
+F 0 "R?" H 3680 3870 50  0000 L CNN
+F 1 "R_Small" H 3680 3810 50  0000 L CNN
+F 2 "" H 3650 3850 60  0000 C CNN
+F 3 "" H 3650 3850 60  0000 C CNN
+	1    3650 3850
+	0    1    1    0
+$EndComp
+Wire Wire Line
+	3150 4000 3550 4000
+Wire Wire Line
+	3550 4000 3550 3850
+Wire Wire Line
+	3750 3850 3900 3850
+$Comp
+L GND #PWR?
+U 1 1 561F3C70
+P 4400 3850
+F 0 "#PWR?" H 4400 3600 50  0001 C CNN
+F 1 "GND" H 4400 3700 50  0000 C CNN
+F 2 "" H 4400 3850 60  0000 C CNN
+F 3 "" H 4400 3850 60  0000 C CNN
+	1    4400 3850
+	0    -1   -1   0
+$EndComp
+Wire Wire Line
+	4300 3850 4400 3850
 $EndSCHEMATC

Commit message: Updated Schematic
Parts:
- added R2: 100K, Resistors_SMD:R_0603, symbol R_Small
- added SW2: SW_PUSH, symbol SW_PUSH
- C1: footprint (none) -> Capacitors_SMD:C_0603
- D1: renamed from D?; footprint (none) -> LEDs:LED-0603
- R1: renamed from R?; value R_Small -> 47; footprint (none) -> Resistors_SMD:R_0603
- gave numbers to parts that had none: 1
Connections:
- wire segments 31 -> 40
Changed lines of the file:
@@
 F 0 "BLE1" H 9650 5300 60  0000 C CNN
 F 1 "BC118" H 9650 5400 60  0000 C CNN
-F 2 "" H 9650 5400 60  0000 C CNN
+F 2 "" H 9650 5400 60  0001 C CNN
 F 3 "" H 9650 5400 60  0000 C CNN
 	1    9900 4200
@@
 $EndComp
 $Comp
-L GND #PWR8
+L GND #PWR01
 U 1 1 560D6740
 P 8350 3050
-F 0 "#PWR8" H 8350 2800 50  0001 C CNN
+F 0 "#PWR01" H 8350 2800 50  0001 C CNN
 F 1 "GND" H 8350 2900 50  0000 C CNN
 F 2 "" H 8350 3050 60  0000 C CNN
@@
 $EndComp
 $Comp
-L +3V3 #PWR1
+L +3V3 #PWR02
 U 1 1 560D743F
 P 800 3300
-F 0 "#PWR1" H 800 3150 50  0001 C CNN
+F 0 "#PWR02" H 800 3150 50  0001 C CNN
 F 1 "+3V3" H 800 3440 50  0000 C CNN
 F 2 "" H 800 3300 60  0000 C CNN
@@
 $EndComp
 $Comp
-L GND #PWR2
+L GND #PWR03
 U 1 1 560D758B
 P 800 4500
-F 0 "#PWR2" H 800 4250 50  0001 C CNN
+F 0 "#PWR03" H 800 4250 50  0001 C CNN
 F 1 "GND" H 800 4350 50  0000 C CNN
 F 2 "" H 800 4500 60  0000 C CNN
@@
 $EndComp
 $Comp
-L +3V3 #PWR9
+L +3V3 #PWR04
 U 1 1 560D7738
 P 8500 4850
-F 0 "#PWR9" H 8500 4700 50  0001 C CNN
+F 0 "#PWR04" H 8500 4700 50  0001 C CNN
 F 1 "+3V3" H 8500 4990 50  0000 C CNN
 F 2 "" H 8500 4850 60  0000 C CNN
@@
 F 0 "C1" H 8560 4620 50  0000 L CNN
 F 1 "10nF" H 8560 4470 50  0000 L CNN
-F 2 "" H 8550 4550 60  0000 C CNN
+F 2 "Capacitors_SMD:C_0603" H 8550 4550 60  0001 C CNN
 F 3 "" H 8550 4550 60  0000 C CNN
 	1    8550 4550
@@
 $EndComp
 $Comp
-L GND #PWR4
+L GND #PWR05
 U 1 1 560D7FCC
 P 4350 4200
-F 0 "#PWR4" H 4350 3950 50  0001 C CNN
+F 0 "#PWR05" H 4350 3950 50  0001 C CNN
 F 1 "GND" H 4350 4050 50  0000 C CNN
 F 2 "" H 4350 4200 60  0000 C CNN
@@
 F 0 "SW1" H 4050 4310 50  0000 C CNN
 F 1 "SW_PUSH" H 3900 4120 50  0000 C CNN
-F 2 "" H 3900 4200 60  0000 C CNN
+F 2 "" H 3900 4200 60  0001 C CNN
 F 3 "" H 3900 4200 60  0000 C CNN
 	1    3900 4200
@@
 F 0 "BT1" H 6450 3950 50  0000 L CNN
 F 1 "Battery" H 6450 3850 50  0000 L CNN
-F 2 "" V 6350 3940 60  0000 C CNN
+F 2 "" V 6350 3940 60  0001 C CNN
 F 3 "" V 6350 3940 60  0000 C CNN
 	1    6350 3900
@@
 $EndComp
 $Comp
-L GND #PWR7
+L GND #PWR06
 U 1 1 560D9BA1
 P 6350 4250
-F 0 "#PWR7" H 6350 4000 50  0001 C CNN
+F 0 "#PWR06" H 6350 4000 50  0001 C CNN
 F 1 "GND" H 6350 4100 50  0000 C CNN
 F 2 "" H 6350 4250 60  0000 C CNN
@@
 $EndComp
 $Comp
-L +3V3 #PWR6
+L +3V3 #PWR07
 U 1 1 560D9BC3
 P 6350 3550
-F 0 "#PWR6" H 6350 3400 50  0001 C CNN
+F 0 "#PWR07" H 6350 3400 50  0001 C CNN
 F 1 "+3V3" H 6350 3690 50  0000 C CNN
 F 2 "" H 6350 3550 60  0000 C CNN
@@
 $EndComp
 $Comp
-L +3V3 #PWR3
+L +3V3 #PWR08
 U 1 1 560DA4CD
 P 3700 3300
-F 0 "#PWR3" H 3700 3150 50  0001 C CNN
+F 0 "#PWR08" H 3700 3150 50  0001 C CNN
 F 1 "+3V3" H 3700 3440 50  0000 C CNN
 F 2 "" H 3700 3300 60  0000 C CNN
@@
 Text GLabel 3550 3600 2    60   Input ~ 0
 WAKE
-Text GLabel 10550 4850 2    60   Input ~ 0
+Text GLabel 10750 4850 2    60   Input ~ 0
 WAKE
 Text GLabel 2850 1950 3    60   Input ~ 0
@@
 P4
 $Comp
-L CONN_01X06 P?
+L CONN_01X06 P1
 U 1 1 561F3005
 P 2900 1750
-F 0 "P?" H 2900 2100 50  0000 C CNN
+F 0 "P1" H 2900 2100 50  0000 C CNN
 F 1 "CONN_01X06" V 3000 1750 50  0000 C CNN
-F 2 "" H 2900 1750 60  0000 C CNN
+F 2 "" H 2900 1750 60  0001 C CNN
 F 3 "" H 2900 1750 60  0000 C CNN
 	1    2900 1750
@@
 	6100 4100 6100 4050
 Wire Wire Line
-	6100 4050 6350 4050
-Wire Wire Line
 	6350 4050 6350 4250
-Text GLabel 6100 3650 1    60   Input ~ 0
-PROG_VIN
-Wire Wire Line
-	6100 3650 6100 3750
-Wire Wire Line
-	6100 3750 6350 3750
 Wire Wire Line
 	6350 3750 6350 3550
@@
 P4
 $Comp
-L LED D?
+L LED D1
 U 1 1 561F3B46
 P 4100 3850
-F 0 "D?" H 4100 3950 50  0000 C CNN
+F 0 "D1" H 4100 3950 50  0000 C CNN
 F 1 "LED" H 4100 3750 50  0000 C CNN
-F 2 "" H 4100 3850 60  0000 C CNN
+F 2 "LEDs:LED-0603" H 4100 3850 60  0001 C CNN
 F 3 "" H 4100 3850 60  0000 C CNN
 	1    4100 3850
@@
 $EndComp
 $Comp
-L R_Small R?
+L R_Small R1
 U 1 1 561F3B97
 P 3650 3850
-F 0 "R?" H 3680 3870 50  0000 L CNN
-F 1 "R_Small" H 3680 3810 50  0000 L CNN
-F 2 "" H 3650 3850 60  0000 C CNN
+F 0 "R1" H 3680 3870 50  0000 L CNN
+F 1 "47" H 3680 3810 50  0000 L CNN
+F 2 "Resistors_SMD:R_0603" H 3650 3850 60  0001 C CNN
 F 3 "" H 3650 3850 60  0000 C CNN
 	1    3650 3850
@@
 	3750 3850 3900 3850
 $Comp
-L GND #PWR?
+L GND #PWR09
 U 1 1 561F3C70
 P 4400 3850
-F 0 "#PWR?" H 4400 3600 50  0001 C CNN
+F 0 "#PWR09" H 4400 3600 50  0001 C CNN
 F 1 "GND" H 4400 3700 50  0000 C CNN
 F 2 "" H 4400 3850 60  0000 C CNN
@@
 Wire Wire Line
 	4300 3850 4400 3850
+Wire Wire Line
+	6100 4050 6350 4050
+Wire Wire Line
+	6100 3650 6100 3750
+Text GLabel 6100 3650 1    60   Input ~ 0
+PROG_VIN
+Wire Wire Line
+	6100 3750 6350 3750
+Wire Wire Line
+	10550 4850 10750 4850
+$Comp
+L R_Small R2
+U 1 1 56303048
+P 10650 5050
+F 0 "R2" H 10680 5070 50  0000 L CNN
+F 1 "100K" H 10680 5010 50  0000 L CNN
+F 2 "Resistors_SMD:R_0603" H 10650 5050 60  0001 C CNN
+F 3 "" H 10650 5050 60  0000 C CNN
+	1    10650 5050
+	1    0    0    -1
+$EndComp
+$Comp
+L GND #PWR010
+U 1 1 563030D2
+P 10650 5250
+F 0 "#PWR010" H 10650 5000 50  0001 C CNN
+F 1 "GND" H 10650 5100 50  0000 C CNN
+F 2 "" H 10650 5250 60  0000 C CNN
+F 3 "" H 10650 5250 60  0000 C CNN
+	1    10650 5250
+	1    0    0    -1
+$EndComp
+Wire Wire Line
+	10650 4950 10650 4850
+Connection ~ 10650 4850
+Wire Wire Line
+	10650 5150 10650 5250
+$Comp
+L GND #PWR011
+U 1 1 56304562
+P 5200 4300
+F 0 "#PWR011" H 5200 4050 50  0001 C CNN
+F 1 "GND" H 5200 4150 50  0000 C CNN
+F 2 "" H 5200 4300 60  0000 C CNN
+F 3 "" H 5200 4300 60  0000 C CNN
+	1    5200 4300
+	0    -1   -1   0
+$EndComp
+$Comp
+L SW_PUSH SW2
+U 1 1 56304568
+P 4750 4300
+F 0 "SW2" H 4900 4410 50  0000 C CNN
+F 1 "SW_PUSH" H 4750 4220 50  0000 C CNN
+F 2 "" H 4750 4300 60  0001 C CNN
+F 3 "" H 4750 4300 60  0000 C CNN
+	1    4750 4300
+	1    0    0    -1
+$EndComp
+Wire Wire Line
+	5050 4300 5200 4300
+Wire Wire Line
+	4450 4300 4150 4300
+Wire Wire Line
+	4150 4300 4150 4350
+Wire Wire Line
+	4150 4350 3700 4350
+Wire Wire Line
+	3700 4350 3700 4300
+Wire Wire Line
+	3700 4300 3150 4300
 $EndSCHEMATC

Commit message: Updated Button code Updated Schematic
Parts:
- removed IC1: ATTINY84A-MM, VQFN20, symbol ATTINY84A-MM
- removed P1: CONN_01X06, symbol CONN_01X06
- added IC1: ATTINY84A-M, war_ic:qfn20, symbol ATTINY84A-M-RESCUE-WAR_Button
- added P2: CONN_02X03, symbol CONN_02X03
- BLE1: footprint (none) -> bc118:bc118
- BT1: footprint (none) -> war_power:20MM_COIN_CELL_SMD
- SW1, SW2: footprint (none) -> Buttons_Switches_ThroughHole:SW_PUSH-12mm
Connections:
- wire segments 40 -> 39
Changed lines of the file:
@@
 EESchema Schematic File Version 2
+LIBS:WAR_Button-rescue
 LIBS:power
 LIBS:device
@@
 $EndDescr
 $Comp
-L ATTINY84A-MM IC1
-U 1 1 560D4AAC
-P 2100 3900
-F 0 "IC1" H 1250 4650 40  0000 C CNN
-F 1 "ATTINY84A-MM" H 2750 3150 40  0000 C CNN
-F 2 "VQFN20" H 2100 3700 35  0000 C CIN
-F 3 "" H 2100 3900 60  0000 C CNN
-	1    2100 3900
-	1    0    0    -1
-$EndComp
-$Comp
 L BC118 BLE1
 U 1 1 560D65FC
@@
 F 0 "BLE1" H 9650 5300 60  0000 C CNN
 F 1 "BC118" H 9650 5400 60  0000 C CNN
-F 2 "" H 9650 5400 60  0001 C CNN
+F 2 "bc118:bc118" H 9650 5400 60  0001 C CNN
 F 3 "" H 9650 5400 60  0000 C CNN
 	1    9900 4200
@@
 F 0 "SW1" H 4050 4310 50  0000 C CNN
 F 1 "SW_PUSH" H 3900 4120 50  0000 C CNN
-F 2 "" H 3900 4200 60  0001 C CNN
+F 2 "Buttons_Switches_ThroughHole:SW_PUSH-12mm" H 3900 4200 60  0001 C CNN
 F 3 "" H 3900 4200 60  0000 C CNN
 	1    3900 4200
@@
 F 0 "BT1" H 6450 3950 50  0000 L CNN
 F 1 "Battery" H 6450 3850 50  0000 L CNN
-F 2 "" V 6350 3940 60  0001 C CNN
+F 2 "war_power:20MM_COIN_CELL_SMD" V 6350 3940 60  0001 C CNN
 F 3 "" V 6350 3940 60  0000 C CNN
 	1    6350 3900
@@
 Text GLabel 10750 4850 2    60   Input ~ 0
 WAKE
-Text GLabel 2850 1950 3    60   Input ~ 0
+Text GLabel 2900 2350 0    60   Input ~ 0
 P1
-Text GLabel 2950 1950 3    60   Input ~ 0
+Text GLabel 2900 2250 0    60   Input ~ 0
 P2
-Text GLabel 3050 1950 3    60   Input ~ 0
+Text GLabel 3400 2350 2    60   Input ~ 0
 P3
-Text GLabel 3150 1950 3    60   Input ~ 0
+Text GLabel 2900 2450 0    60   Input ~ 0
 P4
-$Comp
-L CONN_01X06 P1
-U 1 1 561F3005
-P 2900 1750
-F 0 "P1" H 2900 2100 50  0000 C CNN
-F 1 "CONN_01X06" V 3000 1750 50  0000 C CNN
-F 2 "" H 2900 1750 60  0001 C CNN
-F 3 "" H 2900 1750 60  0000 C CNN
-	1    2900 1750
-	0    -1   -1   0
-$EndComp
-Text GLabel 2600 2250 3    60   Input ~ 0
+Text GLabel 3400 2250 2    60   Input ~ 0
 PROG_VIN
-Text GLabel 2750 2250 3    60   Input ~ 0
+Text GLabel 3400 2450 2    60   Input ~ 0
 PROG_GND
-Wire Wire Line
-	2750 1950 2750 2250
-Wire Wire Line
-	2600 2250 2600 1950
-Wire Wire Line
-	2600 1950 2650 1950
 Text GLabel 6100 4100 3    60   Input ~ 0
 PROG_GND
@@
 F 0 "SW2" H 4900 4410 50  0000 C CNN
 F 1 "SW_PUSH" H 4750 4220 50  0000 C CNN
-F 2 "" H 4750 4300 60  0001 C CNN
+F 2 "Buttons_Switches_ThroughHole:SW_PUSH-12mm" H 4750 4300 60  0001 C CNN
 F 3 "" H 4750 4300 60  0000 C CNN
 	1    4750 4300
@@
 Wire Wire Line
 	3700 4300 3150 4300
+$Comp
+L ATTINY84A-M-RESCUE-WAR_Button IC1
+U 1 1 56304DEF
+P 2100 3900
+F 0 "IC1" H 1250 4650 40  0000 C CNN
+F 1 "ATTINY84A-M" H 2800 3150 40  0000 C CNN
+F 2 "war_ic:qfn20" H 2100 3700 35  0000 C CIN
+F 3 "" H 2100 3900 60  0000 C CNN
+	1    2100 3900
+	1    0    0    -1
+$EndComp
+Wire Wire Line
+	1000 4400 900  4400
+Wire Wire Line
+	900  4400 900  4500
+Connection ~ 900  4500
+$Comp
+L CONN_02X03 P2
+U 1 1 56305C78
+P 3150 2350
+F 0 "P2" H 3150 2550 50  0000 C CNN
+F 1 "CONN_02X03" H 3150 2150 50  0000 C CNN
+F 2 "" H 3150 1150 60  0000 C CNN
+F 3 "" H 3150 1150 60  0000 C CNN
+	1    3150 2350
+	1    0    0    -1
+$EndComp
 $EndSCHEMATC

Commit message: -Finished PCB Design
Parts:
- removed BT1: Battery, war_power:20MM_COIN_CELL_SMD, symbol Battery
- added C1, C2: 4.7uF, Capacitors_SMD:C_0603, symbol C_Small
- added D1: LED, LEDs:LED-0603, symbol LED
- added P1: USB_OTG, war_power:USB_Micro-B, symbol USB_OTG
- added P2: BATT, war_power:JST_2, symbol CONN_01X02
- added P4: RX, Measurement_Points:Measurement_Point_Square-SMD-Pad_Small, symbol CONN_01X01
- added P5: TX, Measurement_Points:Measurement_Point_Square-SMD-Pad_Small, symbol CONN_01X01
- added P6: GND, Measurement_Points:Measurement_Point_Square-SMD-Pad_Small, symbol CONN_01X01
- added P7: BLED1, Measurement_Points:Measurement_Point_Square-SMD-Pad_Small, symbol CONN_01X01
- added P8: BLED2, Measurement_Points:Measurement_Point_Square-SMD-Pad_Small, symbol CONN_01X01
- added Q1: MCP73831, Housings_SOT-23_SOT-143_TSOT-6:SOT-23-5, symbol MCP73831
- added R1: LED_R, Resistors_SMD:R_0603, symbol R_Small
- added R2: PROG, Resistors_SMD:R_0603, symbol R_Small
- P3: renamed from P2; value CONN_02X03 -> HEADER; footprint (none) -> Pin_Headers:Pin_Header_Straight_2x03
- R3: renamed from R1; value 47 -> LED_R
- SW1, SW2: footprint Buttons_Switches_ThroughHole:SW_PUSH-12mm -> Buttons_Switches_SMD:SW_SPST_EVQP2
- renumbered C1 to C3, D1 to D2, R2 to R4
Connections:
- net BLE_RX: now also P4.1 (P1)
- net BLE_TX: now also P5.1 (P1)
- net GND: now also C1.2, C2.1, P1.5 (GND), P2.1 (P1), P6.1 (P1), Q1.2 (VSS), R2.2
- net BLED2: now reaches BLE1.26 (PIO_9)
- net BLED2: now also P8.1 (P1)
- net BLED1: now reaches BLE1.9 (PIO_4)
- net BLED1: now also P7.1 (P1)
- net +3V3 renamed BATT_VCC
- net BATT_VCC: now also C2.2, P2.2 (P2), Q1.3 (VBAT); no longer P3.2 (P2)
- new net: D1.1 (K), Q1.1 (STAT)
- new net: D1.2 (A), R1.2
- new net: Q1.5 (PROG), R2.1
- new net PROG_VCC: C1.1, P1.1 (VCC), P3.2 (P2), Q1.4 (VDD), R1.1
Other:
- moved on the sheet: BLE1, C3, D2, IC1, P3, R3, R4, SW1, SW2
