File: PCB/KiCad_Project/WAR_Button.sch (KiCad schematic (older format))
At the start: 22 parts, among them IC1 ATTINY84A-M, P1 USB_OTG, P2 BATT, P3 HEADER, P4 RX, P5 TX, P6 GND, P7 BLED1, P8 BLED2, Q1 MCP73831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

Commit message: Added MOSFET
Parts:
- added C4: 1uF, Capacitors_SMD:C_0603, symbol C_Small
- added Q2: NTR2101PT1G, Housings_SOT-23_SOT-143_TSOT-6:SOT-23, symbol NTR2101PT1G
- added R5: 100K, Resistors_SMD:R_0603, symbol R_Small
Connections:
- net BATT_VCC: now also Q2.2 (Source); no longer BLE1.17 (VDD_PADS), BLE1.27 (VBAT), C3.2, IC1.5 ((PCINT0/AREF/ADC0)PA0), IC1.9 (VCC)
- net GND: now also C4.1, R5.1
- net PROG_VCC renamed USB_VCC
- net USB_VCC: now also Q2.1 (Gate), R5.2; no longer P3.2 (P2)
- new net LOAD_VCC: BLE1.17 (VDD_PADS), BLE1.27 (VBAT), C3.2, C4.2, IC1.5 ((PCINT0/AREF/ADC0)PA0), IC1.9 (VCC), P3.2 (P2), Q2.3 (Drain)
Other:
- moved on the sheet: C2, D1, Q1, R1, R2
Changed lines of the file:
@@
 L C_Small C2
 U 1 1 563E8DC4
-P 1850 6300
-F 0 "C2" H 1860 6370 50  0000 L CNN
-F 1 "4.7uF" H 1860 6220 50  0000 L CNN
-F 2 "Capacitors_SMD:C_0603" H 1850 6300 60  0001 C CNN
-F 3 "" H 1850 6300 60  0000 C CNN
-	1    1850 6300
+P 2850 6250
+F 0 "C2" H 2860 6320 50  0000 L CNN
+F 1 "4.7uF" H 2860 6170 50  0000 L CNN
+F 2 "Capacitors_SMD:C_0603" H 2850 6250 60  0001 C CNN
+F 3 "" H 2850 6250 60  0000 C CNN
+	1    2850 6250
 	-1   0    0    1
 $EndComp
@@
 L LED D1
 U 1 1 563E8E5E
-P 1700 5800
-F 0 "D1" H 1700 5900 50  0000 C CNN
-F 1 "LED" H 1700 5700 50  0000 C CNN
-F 2 "LEDs:LED-0603" H 1700 5800 60  0001 C CNN
-F 3 "" H 1700 5800 60  0000 C CNN
-	1    1700 5800
+P 2700 5750
+F 0 "D1" H 2700 5850 50  0000 C CNN
+F 1 "LED" H 2700 5650 50  0000 C CNN
+F 2 "LEDs:LED-0603" H 2700 5750 60  0001 C CNN
+F 3 "" H 2700 5750 60  0000 C CNN
+	1    2700 5750
 	-1   0    0    1
 $EndComp
@@
 L R_Small R1
 U 1 1 563E8ED3
-P 1400 5800
-F 0 "R1" H 1430 5820 50  0000 L CNN
-F 1 "LED_R" H 1430 5760 50  0000 L CNN
-F 2 "Resistors_SMD:R_0603" H 1400 5800 60  0001 C CNN
-F 3 "" H 1400 5800 60  0000 C CNN
-	1    1400 5800
+P 2400 5750
+F 0 "R1" H 2430 5770 50  0000 L CNN
+F 1 "LED_R" H 2430 5710 50  0000 L CNN
+F 2 "Resistors_SMD:R_0603" H 2400 5750 60  0001 C CNN
+F 3 "" H 2400 5750 60  0000 C CNN
+	1    2400 5750
 	0    -1   -1   0
 $EndComp
@@
 L MCP73831 Q1
 U 1 1 563E8F3E
-P 2400 5950
-F 0 "Q1" H 2750 6050 40  0000 R CNN
-F 1 "MCP73831" H 3000 5950 40  0000 R TNN
-F 2 "Housings_SOT-23_SOT-143_TSOT-6:SOT-23-5" H 2800 5850 30  0000 C CNN
-F 3 "" H 2450 5950 60  0000 C CNN
-	1    2400 5950
+P 3400 5900
+F 0 "Q1" H 3750 6000 40  0000 R CNN
+F 1 "MCP73831" H 4000 5900 40  0000 R TNN
+F 2 "Housings_SOT-23_SOT-143_TSOT-6:SOT-23-5" H 3800 5800 30  0000 C CNN
+F 3 "" H 3450 5900 60  0000 C CNN
+	1    3400 5900
 	0    1    1    0
 $EndComp
@@
 L GND #PWR08
 U 1 1 563E9261
-P 1950 5950
-F 0 "#PWR08" H 1950 5700 50  0001 C CNN
-F 1 "GND" H 1950 5800 50  0000 C CNN
-F 2 "" H 1950 5950 60  0000 C CNN
-F 3 "" H 1950 5950 60  0000 C CNN
-	1    1950 5950
+P 2950 5900
+F 0 "#PWR08" H 2950 5650 50  0001 C CNN
+F 1 "GND" H 2950 5750 50  0000 C CNN
+F 2 "" H 2950 5900 60  0000 C CNN
+F 3 "" H 2950 5900 60  0000 C CNN
+	1    2950 5900
 	0    1    1    0
 $EndComp
 Text GLabel 1200 4700 3    60   Input ~ 0
 USB_VCC
-Text GLabel 2850 6100 2    60   Input ~ 0
+Text GLabel 3850 6050 2    60   Input ~ 0
 USB_VCC
 $Comp
@@
 L GND #PWR010
 U 1 1 563E9861
-P 1850 6400
-F 0 "#PWR010" H 1850 6150 50  0001 C CNN
-F 1 "GND" H 1850 6250 50  0000 C CNN
-F 2 "" H 1850 6400 60  0000 C CNN
-F 3 "" H 1850 6400 60  0000 C CNN
-	1    1850 6400
+P 2850 6350
+F 0 "#PWR010" H 2850 6100 50  0001 C CNN
+F 1 "GND" H 2850 6200 50  0000 C CNN
+F 2 "" H 2850 6350 60  0000 C CNN
+F 3 "" H 2850 6350 60  0000 C CNN
+	1    2850 6350
 	1    0    0    -1
 $EndComp
@@
 L R_Small R2
 U 1 1 563E9ABE
-P 2850 5550
-F 0 "R2" H 2880 5570 50  0000 L CNN
-F 1 "PROG" H 2880 5510 50  0000 L CNN
-F 2 "Resistors_SMD:R_0603" H 2850 5550 60  0001 C CNN
-F 3 "" H 2850 5550 60  0000 C CNN
-	1    2850 5550
+P 3850 5500
+F 0 "R2" H 3880 5520 50  0000 L CNN
+F 1 "PROG" H 3880 5460 50  0000 L CNN
+F 2 "Resistors_SMD:R_0603" H 3850 5500 60  0001 C CNN
+F 3 "" H 3850 5500 60  0000 C CNN
+	1    3850 5500
 	-1   0    0    1
 $EndComp
@@
 	4100 1300 4100 1350
 Wire Wire Line
-	3150 1100 3700 1100
-Wire Wire Line
 	3550 1400 3150 1400
 Wire Wire Line
@@
 Connection ~ 900  2300
 Wire Wire Line
-	1900 5800 1950 5800
-Wire Wire Line
-	1550 6100 1950 6100
-Wire Wire Line
-	1850 6100 1850 6200
-Wire Wire Line
-	1100 4600 1300 4600
+	2900 5750 2950 5750
+Wire Wire Line
+	2200 6050 2950 6050
+Wire Wire Line
+	2850 6050 2850 6150
 Connection ~ 1200 4600
 Wire Wire Line
-	2850 5800 2850 5650
+	3850 5750 3850 5600
 $Comp
 L GND #PWR011
 U 1 1 563E9C53
-P 2850 5450
-F 0 "#PWR011" H 2850 5200 50  0001 C CNN
-F 1 "GND" H 2850 5300 50  0000 C CNN
-F 2 "" H 2850 5450 60  0000 C CNN
-F 3 "" H 2850 5450 60  0000 C CNN
-	1    2850 5450
+P 3850 5400
+F 0 "#PWR011" H 3850 5150 50  0001 C CNN
+F 1 "GND" H 3850 5250 50  0000 C CNN
+F 2 "" H 3850 5400 60  0000 C CNN
+F 3 "" H 3850 5400 60  0000 C CNN
+	1    3850 5400
 	-1   0    0    1
 $EndComp
@@
 Wire Wire Line
 	2600 4600 2600 4550
-Text GLabel 1550 6100 0    60   Input ~ 0
+Text GLabel 2550 6050 3    60   Input ~ 0
 BATT_VCC
-Connection ~ 1850 6100
-Text GLabel 800  1100 1    60   Input ~ 0
-BATT_VCC
-Text GLabel 8250 2600 0    60   Input ~ 0
-BATT_VCC
-Text GLabel 1300 5800 0    60   Input ~ 0
+Connection ~ 2850 6050
+Text GLabel 2300 5750 0    60   Input ~ 0
 USB_VCC
 Wire Wire Line
 	1200 4350 1200 4700
-Text GLabel 1300 4600 2    60   Input ~ 0
-PROG_VCC
 Wire Wire Line
 	3950 4550 4200 4550
@@
 	4100 4550 4100 4800
 Connection ~ 4100 4550
-Text GLabel 3700 1100 2    60   Input ~ 0
-BATT_VCC
 $Comp
 L CONN_01X01 P4
@@
 Text GLabel 6600 1950 0    60   Input ~ 0
 BLED2
+Text GLabel 950  6150 3    60   Input ~ 0
+LOAD_VCC
+Text GLabel 800  1200 3    60   Input ~ 0
+LOAD_VCC
+Wire Wire Line
+	800  1100 800  1200
+Text GLabel 3500 1100 1    60   Input ~ 0
+LOAD_VCC
+Wire Wire Line
+	3500 1100 3150 1100
+Text GLabel 8250 2600 1    60   Input ~ 0
+LOAD_VCC
+Text GLabel 2200 6400 3    60   Input ~ 0
+USB_VCC
+Wire Wire Line
+	950  6150 1300 6150
+$Comp
+L NTR2101PT1G Q2
+U 1 1 5643C51D
+P 1800 6150
+F 0 "Q2" H 1850 6350 60  0000 C CNN
+F 1 "NTR2101PT1G" H 1850 5950 60  0000 C CNN
+F 2 "Housings_SOT-23_SOT-143_TSOT-6:SOT-23" H 1850 6350 60  0001 C CNN
+F 3 "" H 1850 6350 60  0000 C CNN
+	1    1800 6150
+	-1   0    0    1
+$EndComp
+Wire Wire Line
+	2200 6400 2200 6250
+$Comp
+L C_Small C4
+U 1 1 5644026D
+P 1300 6350
+F 0 "C4" H 1310 6420 50  0000 L CNN
+F 1 "1uF" H 1310 6270 50  0000 L CNN
+F 2 "Capacitors_SMD:C_0603" H 1300 6350 60  0001 C CNN
+F 3 "" H 1300 6350 60  0000 C CNN
+	1    1300 6350
+	-1   0    0    1
+$EndComp
+Wire Wire Line
+	1300 6150 1300 6250
+$Comp
+L GND #PWR015
+U 1 1 56440362
+P 1300 6450
+F 0 "#PWR015" H 1300 6200 50  0001 C CNN
+F 1 "GND" H 1300 6300 50  0000 C CNN
+F 2 "" H 1300 6450 60  0000 C CNN
+F 3 "" H 1300 6450 60  0000 C CNN
+	1    1300 6450
+	1    0    0    -1
+$EndComp
+Text GLabel 1150 6150 1    60   Input ~ 0
+PROG_VCC
+Wire Wire Line
+	1100 4600 1200 4600
+$Comp
+L R_Small R5
+U 1 1 5644486A
+P 2050 6600
+F 0 "R5" H 2080 6620 50  0000 L CNN
+F 1 "100K" H 2080 6560 50  0000 L CNN
+F 2 "Resistors_SMD:R_0603" H 2050 6600 60  0001 C CNN
+F 3 "" H 2050 6600 60  0000 C CNN
+	1    2050 6600
+	-1   0    0    1
+$EndComp
+$Comp
+L GND #PWR016
+U 1 1 56444F96
+P 2050 6700
+F 0 "#PWR016" H 2050 6450 50  0001 C CNN
+F 1 "GND" H 2050 6550 50  0000 C CNN
+F 2 "" H 2050 6700 60  0000 C CNN
+F 3 "" H 2050 6700 60  0000 C CNN
+	1    2050 6700
+	1    0    0    -1
+$EndComp
+Wire Wire Line
+	2050 6500 2050 6350
+Wire Wire Line
+	2050 6350 2200 6350
+Connection ~ 2200 6350
 $EndSCHEMATC

Commit message: Added CONTENTS text file Clarified the schematic for the device.
Parts:
- P3: value HEADER -> PROGRAMMING HEADER
Changed lines of the file:
@@
 P 3700 4450
 F 0 "P3" H 3700 4650 50  0000 C CNN
-F 1 "HEADER" H 3700 4250 50  0000 C CNN
+F 1 "PROGRAMMING HEADER" H 3700 4250 50  0000 C CNN
 F 2 "Pin_Headers:Pin_Header_Straight_2x03" H 3700 3250 60  0001 C CNN
 F 3 "" H 3700 3250 60  0000 C CNN
